File: 2ndOrderLowPass.kicad_sch (KiCad schematic)
At the start: 13 parts, among them U211 LT1169CS8-PBF

Commit message: changed capacitor footprint to match in stock components (0603 to 1206)
Parts:
- C201, C202, C203, C204: footprint Capacitor_SMD:C_0603_1608Metric_Pad1.08x0.95mm_HandSolder -> Capacitor_SMD:C_1206_3216Metric
Changed lines of the file:
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@@
       (effects (font (size 1.27 1.27)))
     )
-    (property "Footprint" "Capacitor_SMD:C_0603_1608Metric_Pad1.08x0.95mm_HandSolder" (at 71.12 79.0448 0)
+    (property "Footprint" "Capacitor_SMD:C_1206_3216Metric" (at 71.12 79.0448 0)
       (effects (font (size 1.27 1.27)) hide)
     )
@@
       (effects (font (size 1.27 1.27)) (justify left))
     )
-    (property "Footprint" "Capacitor_SMD:C_0603_1608Metric_Pad1.08x0.95mm_HandSolder" (at 173.6852 119.38 0)
+    (property "Footprint" "Capacitor_SMD:C_1206_3216Metric" (at 173.6852 119.38 0)
       (effects (font (size 1.27 1.27)) hide)
     )
@@
       (effects (font (size 1.27 1.27)))
     )
-    (property "Footprint" "Capacitor_SMD:C_0603_1608Metric_Pad1.08x0.95mm_HandSolder" (at 184.15 66.3448 0)
+    (property "Footprint" "Capacitor_SMD:C_1206_3216Metric" (at 184.15 66.3448 0)
       (effects (font (size 1.27 1.27)) hide)
     )
@@
       (effects (font (size 1.27 1.27)))
     )
-    (property "Footprint" "Capacitor_SMD:C_0603_1608Metric_Pad1.08x0.95mm_HandSolder" (at 83.82 79.0448 0)
-      (effects (font (size 1.27 1.27)) hide)
-    )
+    (property "Footprint" "Capacitor_SMD:C_1206_3216Metric" (at 83.82 79.0448 0)
+      (effects (font (size 1.27 1.27)) hide)
+    )

Commit message: ToTheEdge,LCSCNums
Moved the 3.5mm connectors to the edge and edited their footprint courtyard so no errors. Adjusted the planes so that it bordered 3.5mm connector pads well and didn't go to edge cuts. Added LCSC part numbers to the parts that were in stock.
Parts:
- 2TP2, 2TP3: LCSC (none) -> C238122
- C201, C202, C203, C204: LCSC (none) -> C2981728
- R211, R212: LCSC (none) -> C351655
- R221, R222: LCSC (none) -> C855838
- R231, R232: LCSC (none) -> C705913
Changed lines of the file:
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@@
       (effects (font (size 1.27 1.27)) (justify bottom) hide)
+    )
+    (property "LCSC" "C238122" (at 207.01 80.01 0)
+      (effects (font (size 1.27 1.27)) hide)
     )
     (pin "TP")
@@
     )
     (property "Datasheet" "~" (at 149.86 82.55 0)
+      (effects (font (size 1.27 1.27)) hide)
+    )
+    (property "LCSC" "C855838" (at 149.86 82.55 0)
       (effects (font (size 1.27 1.27)) hide)
     )
@@
       (effects (font (size 1.27 1.27)) hide)
     )
+    (property "LCSC" "C705913" (at 196.85 105.41 0)
+      (effects (font (size 1.27 1.27)) hide)
+    )
     (pin "1")
     (pin "2")
@@
     (property "Datasheet" "LT1169CS8-PBF" (at 118.11 100.33 0)
       (effects (font (size 1.27 1.27) italic) hide)
+    )
+    (property "LCSC" "" (at 118.11 100.33 0)
+      (effects (font (size 1.27 1.27)) hide)
     )
     (pin "1")
@@
       (effects (font (size 1.27 1.27)) hide)
     )
+    (property "LCSC" "C351655" (at 90.17 87.63 0)
+      (effects (font (size 1.27 1.27)) hide)
+    )
     (pin "1")
     (pin "2")
@@
     )
     (property "Datasheet" "~" (at 67.31 80.01 0)
+      (effects (font (size 1.27 1.27)) hide)
+    )
+    (property "LCSC" "C2981728" (at 67.31 80.01 0)
       (effects (font (size 1.27 1.27)) hide)
     )
@@
       (effects (font (size 1.27 1.27)) hide)
     )
+    (property "LCSC" "C2981728" (at 172.72 115.57 0)
+      (effects (font (size 1.27 1.27)) hide)
+    )
     (pin "1")
     (pin "2")
@@
       (effects (font (size 1.27 1.27)) hide)
     )
+    (property "LCSC" "C351655" (at 95.25 63.5 0)
+      (effects (font (size 1.27 1.27)) hide)
+    )
     (pin "1")
     (pin "2")
@@
     )
     (property "Datasheet" "~" (at 180.34 67.31 0)
+      (effects (font (size 1.27 1.27)) hide)
+    )
+    (property "LCSC" "C2981728" (at 180.34 67.31 0)
       (effects (font (size 1.27 1.27)) hide)
     )
@@
       (effects (font (size 1.27 1.27)) hide)
     )
+    (property "LCSC" "C705913" (at 187.96 119.38 0)
+      (effects (font (size 1.27 1.27)) hide)
+    )
     (pin "1")
     (pin "2")
@@
       (effects (font (size 1.27 1.27)) hide)
     )
+    (property "LCSC" "C855838" (at 165.1 82.55 0)
+      (effects (font (size 1.27 1.27)) hide)
+    )
     (pin "1")
     (pin "2")
@@
     )
     (property "Datasheet" "~" (at 80.01 80.01 0)
+      (effects (font (size 1.27 1.27)) hide)
+    )
+    (property "LCSC" "C2981728" (at 80.01 80.01 0)
       (effects (font (size 1.27 1.27)) hide)
     )
@@
       (effects (font (size 1.27 1.27)) (justify bottom) hide)
     )
+    (property "LCSC" "C238122" (at 129.54 77.47 0)
+      (effects (font (size 1.27 1.27)) hide)
+    )
     (pin "TP")
